File: pcb/3-pin-radio-programmer.brd (EAGLE design)
At the start: 59.7 x 21.6 mm, 14 parts, among them U1 ATTINY85-20SU

Commit message: Adding pull up on reset pin
Parts:
- added R3: 10K, rcl:R0805
Connections:
- net N$11: now also R3.2
- net N$13: now also R3.1
Routing:
- net N$11: track 45.8 -> 47.9 mm
- net N$13: track 23.0 -> 24.6 mm
Changed lines of the file:
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@@
 <attribute name="OC_FARNELL" value="1455164" x="20.32" y="11.43" size="1.778" layer="27" display="off"/>
 </element>
+<element name="R3" library="rcl" package="R0805" value="10K" x="15.24" y="15.24" rot="R180"/>
 </elements>
 <signals>
@@
 <wire x1="2.54" y1="13.55" x2="5.5" y2="16.51" width="0.4064" layer="1"/>
 <wire x1="5.5" y1="16.51" x2="7.62" y2="16.51" width="0.4064" layer="1"/>
-<wire x1="7.62" y1="16.51" x2="20.8534" y2="16.51" width="0.4064" layer="1"/>
+<wire x1="7.62" y1="16.51" x2="12.7" y2="16.51" width="0.4064" layer="1"/>
+<wire x1="12.7" y1="16.51" x2="20.8534" y2="16.51" width="0.4064" layer="1"/>
 <wire x1="20.8534" y1="16.51" x2="24.0284" y2="13.335" width="0.4064" layer="1"/>
 <wire x1="29.21" y1="13.97" x2="24.6634" y2="13.97" width="0.4064" layer="1"/>
@@
 <wire x1="35.56" y1="15.24" x2="36.83" y2="13.97" width="0.4064" layer="1"/>
 <wire x1="36.83" y1="13.97" x2="36.83" y2="6.35" width="0.4064" layer="1"/>
+<contactref element="R3" pad="2"/>
+<wire x1="14.29" y1="15.24" x2="13.97" y2="15.24" width="0.4064" layer="1"/>
+<wire x1="13.97" y1="15.24" x2="12.7" y2="16.51" width="0.4064" layer="1"/>
 </signal>
 <signal name="N$13">
@@
 <wire x1="17.78" y1="15.24" x2="17.78" y2="14.5034" width="0.4064" layer="1"/>
 <wire x1="17.78" y1="14.5034" x2="16.6116" y2="13.335" width="0.4064" layer="1"/>
+<contactref element="R3" pad="1"/>
+<wire x1="16.19" y1="15.24" x2="17.78" y2="15.24" width="0.4064" layer="1"/>
 </signal>
 <signal name="N$5">
